Commit message: Add Ares control demos and state machine

File: model/Ares/urdf/Ares.urdf (robot description, URDF)
Before this commit: robot Ares, 13 links, 12 joints
Joints:
- joint lb_calf_thigh_joint: limit lower=-3.14 upper=3.14 effort=17 velocity=300 -> lower=-1.65 upper=-0.13 effort=17 velocity=300
- joint lb_hip_base_joint: limit lower=-3.14 upper=3.14 effort=17 velocity=300 -> lower=-1.57 upper=0.5 effort=17 velocity=300
- joint lb_thigh_hip_joint: limit lower=-3.14 upper=3.14 effort=17 velocity=300 -> lower=-2.35 upper=2.35 effort=17 velocity=300
- joint lf_calf_thigh_joint: limit lower=-3.14 upper=3.14 effort=17 velocity=300 -> lower=-0.9 upper=0.75 effort=17 velocity=300
- joint lf_hip_base_joint: limit lower=-3.14 upper=3.14 effort=17 velocity=300 -> lower=-0.5 upper=1.57 effort=17 velocity=300
- joint lf_thigh_hip_joint: limit lower=-3.14 upper=3.14 effort=17 velocity=300 -> lower=-2.35 upper=2.35 effort=17 velocity=300
- joint rb_calf_thigh_joint: limit lower=-3.14 upper=3.14 effort=17 velocity=300 -> lower=-0.45 upper=1.35 effort=17 velocity=300
- joint rb_hip_base_joint: limit lower=-3.14 upper=3.14 effort=17 velocity=300 -> lower=-0.5 upper=1.57 effort=17 velocity=300
- joint rb_thigh_hip_joint: limit lower=-3.14 upper=3.14 effort=17 velocity=300 -> lower=-2.35 upper=2.35 effort=17 velocity=300
- joint rf_calf_thigh_joint: limit lower=-3.14 upper=3.14 effort=17 velocity=300 -> lower=-0.7 upper=0.9 effort=17 velocity=300
- joint rf_hip_base_joint: limit lower=-3.14 upper=3.14 effort=17 velocity=300 -> lower=-1.57 upper=0.5 effort=17 velocity=300
- joint rf_thigh_hip_joint: limit lower=-3.14 upper=3.14 effort=17 velocity=300 -> lower=-2.35 upper=2.35 effort=17 velocity=300
